File: hardware/LPC1114-LCD.kicad_sch (KiCad schematic)
At the start: 58 parts, among them J1 USB_B_Micro, J2 SWD, J3 UART, Q1 BC337, Q2 BC337, SW1 MODE/ISP, SW2 UP, SW3 DOWN, SW4 OK, SW5 RESET, U1 LPC1114FN28/102, U2 MCP1700-3302E/TO, U3 CH340C, U4 DS3231MZ+, Y1 12MHz

Commit message: Hardware v1.1: JLCPCB PCBA with Basic parts, Pomodoro timer, 80x52 mm
- Main use is now a Pomodoro timer: RTC (DS3231M) and CR2032 removed,
  timekeeping from the 12 MHz crystal; PTC fuse removed
- SMD redesign for JLCPCB assembly: 0603/0805 passives and LEDs,
  XC6206 LDO, SS8050, B5819W, 3225 crystal, TS-1187A buttons (all Basic);
  CH340C and micro USB are the only Extended parts
- User-soldered: LPC1114 (+socket), LCD, 10k multiturn trimmer,
  TDK PS1420P02CT piezo buzzer, USBLC6-2SC6, J2 (1x7 SWD+I2C) and
  J3 (1x3 UART) pads
- PCB reduced from 80x76 to 80x52 mm; ERC/DRC clean, parity OK, fully routed
- JLCPCB BOM + CPL and hand-solder list generated by export_fab.ps1
- Enclosure updated: 92.8x64.8x31.4 mm, longer button stems, LED light pipes
- Docs: schematic review for JLCPCB, design notes, README, board.h

Co-Authored-By: Claude Opus 5.5 <noreply@anthropic.com>
Parts:
- removed BT1: CR2032, Battery:BatteryHolder_MYOUNG_BS-07-A1BJ001_CR2032, symbol Device:Battery_Cell
- removed C9: 100nF, Capacitor_THT:C_Disc_D3.0mm_W1.6mm_P2.50mm, symbol Device:C
- removed D5: 1N4148, Diode_THT:D_DO-35_SOD27_P2.54mm_Vertical_AnodeUp, symbol Device:D
- removed F1: 500mA, Fuse:Fuse_1206_3216Metric_Pad1.42x1.75mm_HandSolder, symbol Device:Polyfuse
- removed H1, H2: M3, MountingHole:MountingHole_3.2mm_M3, symbol Mechanical:MountingHole
- removed RN1: 10k, Resistor_THT:R_Array_SIP7, symbol Device:R_Network06
- removed U4: DS3231MZ+, Package_SO:SOIC-8_3.9x4.9mm_P1.27mm, symbol Timer_RTC:DS3231MZ
- added R16: 1k, Resistor_SMD:R_0603_1608Metric, symbol Device:R
- added U5: USBLC6-2SC6, Package_TO_SOT_SMD:SOT-23-6_Handsoldering, symbol Power_Protection:USBLC6-2SC6
- BZ1: value Passive buzzer -> PS1420P02CT; footprint Buzzer_Beeper:Buzzer_12x9.5RM7.6 -> LPC1114-LCD:Buzzer_TDK_PS1420P02CT_D14mm_P10mm; Assembly (none) -> USER; MPN 12x9.5mm passive magnetic buzzer 5V (e.g. TMB12A05 / 12085) -> TDK PS1420P02CT (piezo, D14 mm, pitch 10 mm)
- C1, C2: footprint Capacitor_THT:C_Disc_D5.0mm_W2.5mm_P5.00mm -> Capacitor_SMD:C_0805_2012Metric; LCSC (none) -> C15850; MPN 10uF 25V X5R radial MLCC P5.08 -> (none)
- C10, C3, C4, C7, C8: footprint Capacitor_THT:C_Disc_D3.0mm_W1.6mm_P2.50mm -> Capacitor_SMD:C_0603_1608Metric; LCSC (none) -> C14663
- C5, C6: value 18pF -> 33pF; footprint Capacitor_THT:C_Disc_D3.0mm_W1.6mm_P2.50mm -> Capacitor_SMD:C_0603_1608Metric; LCSC (none) -> C1663
- D1: footprint LED_THT:LED_D3.0mm -> LED_SMD:LED_0805_2012Metric; LCSC (none) -> C84256
- D2: footprint LED_THT:LED_D3.0mm -> LED_SMD:LED_0805_2012Metric; LCSC (none) -> C2296
- D3, D4: footprint LED_THT:LED_D3.0mm -> LED_SMD:LED_0805_2012Metric; LCSC (none) -> C2297
- D6, D7: value BAT43 -> B5819W; footprint Diode_THT:D_DO-35_SOD27_P2.54mm_Vertical_AnodeUp -> Diode_SMD:D_SOD-123; LCSC (none) -> C8598
- DS1, J3, RV1, U1: Assembly (none) -> USER
- J1: footprint Connector_USB:USB_Micro-B_Wuerth_629105150521 -> Connector_USB:USB_Micro-B_XKB_U254-051T-4BH83-F1S; LCSC (none) -> C397452; MPN Wurth 629105150521 -> XKB U254-051T-4BH83-F1S
- J2: value SWD -> SWD+I2C; footprint Connector_IDC:IDC-Header_2x05_P2.54mm_Vertical -> Connector_PinHeader_2.54mm:PinHeader_1x07_P2.54mm_Vertical; symbol Connector:Conn_ARM_JTAG_SWD_10 -> Connector_Generic:Conn_01x07; Assembly (none) -> USER
- Q1, Q2: value BC337 -> SS8050; footprint Package_TO_SOT_THT:TO-92_Inline_Wide -> Package_TO_SOT_SMD:SOT-23; symbol Transistor_BJT:BC337 -> Transistor_BJT:Q_NPN_BEC; LCSC (none) -> C2150
- R1, R13, R15: footprint Resistor_THT:R_Axial_DIN0207_L6.3mm_D2.5mm_P2.54mm_Vertical -> Resistor_SMD:R_0603_1608Metric; LCSC (none) -> C25804
- R10, R11, R9: footprint Resistor_THT:R_Axial_DIN0207_L6.3mm_D2.5mm_P2.54mm_Vertical -> Resistor_SMD:R_0603_1608Metric; LCSC (none) -> C22775
- R12, R14, R2, R8: footprint Resistor_THT:R_Axial_DIN0207_L6.3mm_D2.5mm_P2.54mm_Vertical -> Resistor_SMD:R_0603_1608Metric; LCSC (none) -> C21190
- R3, R4: footprint Resistor_THT:R_Axial_DIN0207_L6.3mm_D2.5mm_P2.54mm_Vertical -> Resistor_SMD:R_0603_1608Metric; LCSC (none) -> C23162
- R5, R6, R7: footprint Resistor_THT:R_Axial_DIN0207_L6.3mm_D2.5mm_P2.54mm_Vertical -> Resistor_SMD:R_0603_1608Metric; LCSC (none) -> C23179
- RN2: footprint Resistor_THT:R_Array_SIP5 -> Resistor_SMD:R_Array_Convex_4x0603; symbol Device:R_Network04 -> Device:R_Pack04; LCSC (none) -> C29718
- SW1, SW2, SW3, SW4, SW5: footprint Button_Switch_THT:SW_PUSH_6mm -> LPC1114-LCD:SW_TS-1187A_5.1x5.1mm; LCSC (none) -> C318884
- U2: value MCP1700-3302E/TO -> XC6206P332MR-G; footprint Package_TO_SOT_THT:TO-92_Inline_Wide -> Package_TO_SOT_SMD:SOT-23; symbol Regulator_Linear:MCP1700x-330xxTO -> Regulator_Linear:XC6206PxxxMR; LCSC (none) -> C5446; MPN Microchip MCP1700-3302E/TO -> Torex XC6206P332MR-G
- U3: LCSC (none) -> C84681
- Y1: footprint Crystal:Crystal_HC49-4H_Vertical -> Crystal:Crystal_SMD_3225-4Pin_3.2x2.5mm; symbol Device:Crystal -> Device:Crystal_GND24; LCSC (none) -> C9002; MPN 12 MHz HC-49/S, CL=18pF -> YXC X322512MSB4SI 12MHz CL=20pF
Connections:
- net VBUS is gone; now on net +5V: J1.1 (VBUS)
- net +3V3: now also RN2.5 (R4.2), RN2.6 (R3.2), RN2.7 (R2.2), RN2.8 (R1.2), U2.2 (VO); no longer RN2.1 (common), U2.3 (VO)
- net +5V: now also U2.3 (VI), R16.1, U5.5 (VBUS); no longer U2.2 (VI)
- net BTN_DOWN: now also RN2.3 (R3.1); no longer RN2.4 (R3)
- net BTN_MODE: now also RN2.1 (R1.1); no longer RN2.2 (R1)
- net BTN_OK: now also RN2.4 (R4.1); no longer RN2.5 (R4)
- net BTN_UP: now also RN2.2 (R2.1); no longer RN2.3 (R2)
- net BUZ_K: now also Q2.3 (C), R16.2; no longer Q2.1 (C)
- net GND: now also Q1.2 (E), Q2.2 (E), Y1.2 (G), Y1.4 (G), U5.2 (GND); no longer J2.3 (GND), J2.9 (GNDDetect), Q1.3 (E), Q2.3 (E)
- net I2C_SCL: now also J2.6 (Pin_6)
- net I2C_SDA: now also J2.7 (Pin_7)
- net LCD_K: now also Q1.3 (C); no longer Q1.1 (C)
- net SWCLK: now also J2.3 (Pin_3); no longer J2.4 (SWCLK/TCK)
- net USB_DM: now also U5.3 (I/O2), U5.4 (I/O2)
- net USB_DP: now also U5.1 (I/O1), U5.6 (I/O1)
- net XTAL_OUT: now also Y1.3; no longer Y1.2
- net nRESET: now also J2.4 (Pin_4); no longer J2.10 (~{RESET})
- net at R14.2: now also Q2.1 (B); no longer Q2.2 (B)
- net at R12.2: now also Q1.1 (B); no longer Q1.2 (B)
- no-connect marks 18 -> 12
Other:
- note added: "Assembly=USER parts (U1, DS1, RV1, BZ1, U5, J2, J3) are hand-soldered; all others are JLCPCB PCBA (LCSC field)."
- note added: "HEADERS (pads only): SWD + I2C, UART"
- note added: "LCD R/W tied to GND (write-only). RS/E/D4-D7 driven push-pull at 3.3V (HD44780/ST7066 VIH = 2.2V)."
- note added: "MCU LPC1114FN28 (DIP28) + 12MHz + RESET + BUZZER"
- note added: "PIO0_4/PIO0_5 (I2C) on J2 pins 6/7 for expansion modules."
- note added: "POWER: USB 5V (ESD) -> 3.3V LDO"
- note removed: "LCD R/W tied to GND (write-only). RS/E/D4-D7 can be push-pull 3.3V or open-drain with RN1 pull-ups to 5V."
- note removed: "MCU LPC1114FN28 (DIP28) + 12MHz + SWD + RESET + BUZZER"
- note removed: "POWER: USB 5V -> 3.3V LDO"
- note removed: "RTC (DS3231MZ) + CR2032 backup"
- title: LPC1114-LCD - Digital clock board -> LPC1114-LCD - Pomodoro timer / clock
- moved on the sheet: C5, C6, J3, R3, R4, U2

Commit message: Hardware v1.2: optional RTC (DNP), USBLC6 bypass and UART source selection
- Optional RTC on the bottom side, marked DNP: DS3231MZ+ (U4) between the
  DIP rows, C9 and a Keystone 3034 SMD CR2032 holder (BT1) on the J2 I2C bus;
  excluded from the JLCPCB BOM/CPL, listed in LPC1114-LCD_DNP_options.csv
- USB D+/D- now flow through U5 (USBLC6-2SC6); JP3/JP4 (bottom, open)
  bypass it when U5 is not fitted
- UART source selection: JP5/JP6 3-pad jumpers (bottom), 1-2 CH340
  (bridged by default), 2-3 external UART on J3, so both never connect together
- ERC/DRC clean, schematic parity OK (DNP attributes), fully connected
- Enclosure: 1 mm base pocket for the optional battery holder
- Docs: jumper configuration table, design notes, README, board.h

Co-Authored-By: Claude Opus 5.5 <noreply@anthropic.com>
Parts:
- added BT1: CR2032, Battery:BatteryHolder_Keystone_3034_1x20mm, symbol Device:Battery_Cell
- added C9: 100nF, Capacitor_SMD:C_0603_1608Metric, symbol Device:C
- added JP3: BYP_D+, Jumper:SolderJumper-2_P1.3mm_Open_Pad1.0x1.5mm, symbol Jumper:SolderJumper_2_Open
- added JP4: BYP_D-, Jumper:SolderJumper-2_P1.3mm_Open_Pad1.0x1.5mm, symbol Jumper:SolderJumper_2_Open
- added JP5: RX_SEL, Jumper:SolderJumper-3_P1.3mm_Bridged12_Pad1.0x1.5mm, symbol Jumper:SolderJumper_3_Bridged12
- added JP6: TX_SEL, Jumper:SolderJumper-3_P1.3mm_Bridged12_Pad1.0x1.5mm, symbol Jumper:SolderJumper_3_Bridged12
- added U4: DS3231MZ+, Package_SO:SOIC-8_3.9x4.9mm_P1.27mm, symbol Timer_RTC:DS3231MZ
Connections:
- net +3V3: now also C9.1, U4.2 (VCC)
- net GND: now also BT1.2 (-), C9.2, U4.5 (GND)
- net I2C_SCL: now also U4.8 (SCL)
- net I2C_SDA: now also U4.7 (SDA)
- net UART_RXD: now also JP5.2 (C); no longer J3.2 (Pin_2), R2.1
- net UART_TXD: now also JP6.2 (C); no longer J3.3 (Pin_3), U3.3 (RXD)
- net USB_DM: now also JP4.2 (B); no longer J1.2 (D-), U5.3 (I/O2)
- net USB_DP: now also JP3.2 (B); no longer J1.3 (D+), U5.1 (I/O1)
- new net CH340_RXD: JP6.1 (A), U3.3 (RXD)
- new net CH340_TXD_R: JP5.1 (A), R2.1
- new net EXT_RXD: J3.2 (Pin_2), JP5.3 (B)
- new net EXT_TXD: J3.3 (Pin_3), JP6.3 (B)
- new net USB_DM_C: J1.2 (D-), JP4.1 (A), U5.3 (I/O2)
- new net USB_DP_C: J1.3 (D+), JP3.1 (A), U5.1 (I/O1)
- new net VBAT: BT1.1 (+), U4.6 (VBAT)
- no-connect marks 12 -> 15
Other:
- note added: "Assembly=USER parts (U1, DS1, RV1, BZ1, U5, J2, J3) are hand-soldered; DNP parts are not fitted; the rest is JLCPCB PCBA."
- note added: "HEADERS (pads) + OPTIONAL RTC (bottom side, DNP)"
- note added: "I2C on J2 pins 6/7. U4/C9/BT1 = optional RTC, bottom side, DNP."
- note added: "JP3/JP4: bridge only if U5 is not fitted. JP5/JP6: 1-2 = CH340 (default), 2-3 = external UART on J3."
- note removed: "Assembly=USER parts (U1, DS1, RV1, BZ1, U5, J2, J3) are hand-soldered; all others are JLCPCB PCBA (LCSC field)."
- note removed: "HEADERS (pads only): SWD + I2C, UART"
- note removed: "PIO0_4/PIO0_5 (I2C) on J2 pins 6/7 for expansion modules."
- moved on the sheet: J2, J3
